Commit message: Camera and gripper working in gazebo

File: src/erobotics_description/urdf/adaptative_gripper.urdf.xacro (robot description, xacro)
@@ -47,4 +47,18 @@
       <mimic joint="gripper_controller" multiplier="1.0" offset="0" />
     </joint>
+  <!-- Definición de ros2_control para el Gripper -->
+    <!-- Articulación Maestra del Gripper -->
+  <ros2_control name="GazeboSimSystem" type="system">
+    <hardware>
+      <plugin>gz_ros2_control/GazeboSimSystem</plugin>
+    </hardware>
+      <joint name="gripper_controller">
+        <command_interface name="position"/>
+        <state_interface name="position">
+          <param name="initial_value">0.0</param>
+        </state_interface>
+        <state_interface name="velocity"/>
+      </joint>
+  </ros2_control>
   </xacro:macro>
 </robot>

File: src/erobotics_description/urdf/erobotics_ros2_control.xacro (robot description, xacro)
@@ -56,12 +56,4 @@
       <state_interface name="velocity"/>
     </joint>
-    <!-- Articulación Maestra del Gripper -->
-    <joint name="gripper_controller">
-      <command_interface name="position"/>
-      <state_interface name="position">
-        <param name="initial_value">0.0</param>
-      </state_interface>
-      <state_interface name="velocity"/>
-    </joint>
   </ros2_control>
   <!-- Configuraciones visuales adicionales para Gazebo -->

File: src/erobotics_description/urdf/mycobot_280_arduino.urdf.xacro (robot description, xacro)
@@ -75,5 +75,5 @@
   <xacro:if value="$(arg use_camera)">
     <xacro:rgb_camera parent="joint6" prefix="robot">
-      <origin xyz="0.03 0 0.02" rpy="0 0 0"/>
+      <origin xyz="0.03 0 0.02" rpy="0 0 -${pi/2}"/>
     </xacro:rgb_camera>
   </xacro:if>
